Commit message: urdf: fix x center position

File: urdf/explorer.urdf (robot description, URDF)
Before this commit: robot explorer, 6 links, 5 joints
Links:
- removed link scan
- added link forward_sensor; visual box size=0.015 0.045 0.03
Joints:
- removed joint scan_joint
- added joint forward_sensor_joint: type fixed, parent base_link, child forward_sensor, origin xyz=0.07 0 0.06 rpy=0 0 0
- joint aft_wheel_joint: origin xyz=0 0 0.005 rpy=1.57 0 0 -> xyz=0 0 -0.0475 rpy=1.57 0 0
- joint left_wheel_joint: origin xyz=0.07 -0.08 0.026 rpy=1.57 0 0 -> xyz=0 -0.08 0.026 rpy=1.57 0 0
- joint right_wheel_joint: origin xyz=0.07 0.08 0.026 rpy=1.57 0 0 -> xyz=0 0.08 0.026 rpy=1.57 0 0
- joint tail_joint: origin xyz=-0.04 0 0.005 rpy=0 0 0 -> xyz=-0.1 0 0.0575 rpy=0 0 0

Commit message: Migration to ros control (diff_drive_controller)

File: urdf/explorer.urdf (robot description, URDF)
Before this commit: robot explorer, 6 links, 5 joints
Links:
- link left_wheel: geometry collision cylinder length=0.02 radius=0.026; visual cylinder length=0.02 radius=0.026
- link right_wheel: geometry collision cylinder length=0.02 radius=0.026; visual cylinder length=0.02 radius=0.026
